Commit message: with line world

File: Gazebo/catkin_ws/src/mybot_description/urdf/macros.xacro (robot description, xacro)
@@ -1,25 +1,27 @@
 <?xml version="1.0"?>
-<robot xmlns:xacro="http://www.ros.org/wiki/xacro" name="mybot">
-      <xacro:macro name="cylinder_inertia" params="m r h">
+<robot>
+     <macro name="cylinder_inertia" params="m r h">
         <inertia  ixx="${m*(3*r*r+h*h)/12}" ixy = "0" ixz = "0"
                   iyy="${m*(3*r*r+h*h)/12}" iyz = "0"
                   izz="${m*r*r/2}" />
-      </xacro:macro>
-      <xacro:macro name="box_inertia" params="m x y z">
+      </macro>
+      <macro name="box_inertia" params="m x y z">
         <inertia  ixx="${m*(y*y+z*z)/12}" ixy = "0" ixz = "0"
                   iyy="${m*(x*x+z*z)/12}" iyz = "0"
                   izz="${m*(x*x+z*z)/12}" />
-      </xacro:macro>
-      <xacro:macro name="sphere_inertia" params="m r">
+      </macro>
+      <macro name="sphere_inertia" params="m r">
         <inertia  ixx="${2*m*r*r/5}" ixy = "0" ixz = "0"
                   iyy="${2*m*r*r/5}" iyz = "0"
                   izz="${2*m*r*r/5}" />
-      </xacro:macro>
-	<xacro:macro name="wheel" params="lr tY"><link name="${lr}_wheel">
-		<collision>
-		<origin xyz="0 0 0" rpy="0 ${PI/2} ${PI/2}" /><geometry>
-        	<cylinder length="${wheelWidth}" radius="${wheelRadius}"/>
-        	</geometry>
-        	</collision>
+      </macro>
+     <macro name="wheel" params="lr tY">
+       <link name="${lr}_wheel">
+        <collision>
+          <origin xyz="0 0 0" rpy="0 ${PI/2} ${PI/2}" />
+          <geometry>
+           <cylinder length="${wheelWidth}" radius="${wheelRadius}"/>
+          </geometry>
+        </collision>
         <visual>
           <origin xyz="0 0 0" rpy="0 ${PI/2} ${PI/2}" />
@@ -50,9 +52,10 @@
           <limit effort="100" velocity="100"/>
           <joint_properties damping="0.0" friction="0.0"/>
+	  <hardwareInterface>EffortJointInterface</hardwareInterface>
         </joint>
       <transmission name="${lr}_trans">
         <type>transmission_interface/SimpleTransmission</type>
         <joint name="${lr}_wheel_hinge">
-		<hardwareInterface>EffortJointInterface</hardwareInterface>
+	  <hardwareInterface>EffortJointInterface</hardwareInterface>
 	</joint>
         <actuator name="${lr}Motor">
@@ -61,19 +64,4 @@
         </actuator>
       </transmission>
-     </xacro:macro>
-     <xacro:macro name="cylinder_inertia" params="m r h">
-        <inertia  ixx="${m*(3*r*r+h*h)/12}" ixy = "0" ixz = "0"
-                  iyy="${m*(3*r*r+h*h)/12}" iyz = "0"
-                  izz="${m*r*r/2}" />
-      </xacro:macro>
-      <xacro:macro name="box_inertia" params="m x y z">
-        <inertia  ixx="${m*(y*y+z*z)/12}" ixy = "0" ixz = "0"
-                  iyy="${m*(x*x+z*z)/12}" iyz = "0"
-                  izz="${m*(x*x+z*z)/12}" />
-      </xacro:macro>
-      <xacro:macro name="sphere_inertia" params="m r">
-        <inertia  ixx="${2*m*r*r/5}" ixy = "0" ixz = "0"
-                  iyy="${2*m*r*r/5}" iyz = "0"
-                  izz="${2*m*r*r/5}" />
-      </xacro:macro>
+     </macro>
 </robot>

File: Gazebo/catkin_ws/src/mybot_description/urdf/mybot.xacro (robot description, xacro)
@@ -1,4 +1,4 @@
 <?xml version="1.0"?>
-<robot xmlns:xacro="http://www.ros.org/wiki/xacro" name="mybot">
+<robot name="mybot" xmlns:xacro="http://www.ros.org/wiki/xacro">
   <xacro:property name="PI" value="3.1415926535897931"/>
   <xacro:property name="chassisHeight" value="0.1"/>
