Commit message: line sensors added

File: Gazebo/catkin_ws/src/mybot_description/urdf/mybot.xacro (robot description, xacro)
@@ -14,4 +14,8 @@
   <xacro:property name="cameraSize" value="0.05"/>
   <xacro:property name="cameraMass" value="0.1"/>
+  <xacro:property name="cameraAngle" value="20"/>
+  <xacro:property name="sensorSize" value="0.01"/>
+  <xacro:property name="sensorAngle" value="45"/>
+  <xacro:property name="sensorSpacing" value="0.04"/>
   <xacro:include filename="$(find mybot_description)/urdf/mybot.gazebo" />
   <xacro:include filename="$(find mybot_description)/urdf/materials.xacro" />
@@ -68,5 +72,5 @@
   <wheel lr="right" tY="1"/>
   <joint name="camera_joint" type="fixed">
-    <origin xyz="${-cameraSize+chassisLength/2} 0 ${cameraSize+wheelRadius+cameraSize/2}" rpy="0 0 0"/>
+    <origin xyz="${cameraSize+chassisLength/2} 0 ${cameraSize+wheelRadius+cameraSize/2}" rpy="0 ${cameraAngle} 0"/>
     <parent link="chassis"/>
     <child link="camera"/>
@@ -74,5 +78,5 @@
   <link name="camera">
     <collision>
-      <origin xyz="0 0 0" rpy="0 0 0"/>
+      <origin xyz="${cameraSize} 0 0" rpy="0 0 0"/>
       <geometry>
 	<box size="${cameraSize} ${cameraSize} ${cameraSize}"/>
@@ -80,5 +84,5 @@
     </collision>
     <visual>
-      <origin xyz="0 0 0" rpy="0 0 0"/>
+      <origin xyz="0 0 0" rpy="0 ${cameraAngle} 0"/>
       <geometry>
 	<box size="${cameraSize} ${cameraSize} ${cameraSize}"/>
@@ -92,3 +96,211 @@
     </inertial>
   </link>
+<!--/////////////////////////////////////////////////////////////////-->
+  <joint name="left_sensor1" type="fixed">
+    <origin xyz="${chassisLength/2} ${sensorSpacing} ${wheelRadius/2}" rpy="0 ${sensorAngle} 0"/>
+    <parent link="chassis"/>
+    <child link="l_sensor_1"/>
+  </joint>
+  <link name="l_sensor_1">
+    <collision>
+      <origin xyz="0 0 0" rpy="0 ${sensorAngle} 0"/>
+      <geometry>
+	<box size="${sensorSize} ${sensorSize} ${sensorSize}"/>
+      </geometry>
+    </collision>
+    <visual>
+      <origin xyz="0 0 0" rpy="0 ${sensorAngle} 0"/>
+      <geometry>
+	<box size="${sensorSize} ${sensorSize} ${sensorSize}"/>
+      </geometry>
+      <material name="blue"/>
+    </visual>
+    <inertial>
+      <mass value="${cameraMass}" />
+      <origin xyz="0 0 0" rpy="0 0 0"/>
+      <box_inertia m="${cameraMass}" x="${sensorSize}" y="${sensorSize}" z="${sensorSize}" />
+    </inertial>
+  </link>
+<!--/////////////////////////////////////////////////////////////////-->
+  <joint name="right_sensor1" type="fixed">
+    <origin xyz="${chassisLength/2} ${-sensorSpacing} ${wheelRadius/2}" rpy="0 ${sensorAngle} 0"/>
+    <parent link="chassis"/>
+    <child link="r_sensor_1"/>
+  </joint>
+  <link name="r_sensor_1">
+    <collision>
+      <origin xyz="0 0 0" rpy="0 ${sensorAngle} 0"/>
+      <geometry>
+	<box size="${sensorSize} ${sensorSize} ${sensorSize}"/>
+      </geometry>
+    </collision>
+    <visual>
+      <origin xyz="0 0 0" rpy="0 ${sensorAngle} 0"/>
+      <geometry>
+	<box size="${sensorSize} ${sensorSize} ${sensorSize}"/>
+      </geometry>
+      <material name="blue"/>
+    </visual>
+    <inertial>
+      <mass value="${cameraMass}" />
+      <origin xyz="0 0 0" rpy="0 0 0"/>
+      <box_inertia m="${cameraMass}" x="${sensorSize}" y="${sensorSize}" z="${sensorSize}" />
+    </inertial>
+  </link>
+<!--/////////////////////////////////////////////////////////////////-->
+  <joint name="left_sensor2" type="fixed">
+    <origin xyz="${chassisLength/2} ${2*sensorSpacing} ${wheelRadius/2}" rpy="0 ${sensorAngle} 0"/>
+    <parent link="chassis"/>
+    <child link="l_sensor_2"/>
+  </joint>
+  <link name="l_sensor_2">
+    <collision>
+      <origin xyz="0 0 0" rpy="0 ${sensorAngle} 0"/>
+      <geometry>
+	<box size="${sensorSize} ${sensorSize} ${sensorSize}"/>
+      </geometry>
+    </collision>
+    <visual>
+      <origin xyz="0 0 0" rpy="0 ${sensorAngle} 0"/>
+      <geometry>
+	<box size="${sensorSize} ${sensorSize} ${sensorSize}"/>
+      </geometry>
+      <material name="blue"/>
+    </visual>
+    <inertial>
+      <mass value="${cameraMass}" />
+      <origin xyz="0 0 0" rpy="0 0 0"/>
+      <box_inertia m="${cameraMass}" x="${sensorSize}" y="${sensorSize}" z="${sensorSize}" />
+    </inertial>
+  </link>
+<!--/////////////////////////////////////////////////////////////////-->
+  <joint name="right_sensor2" type="fixed">
+    <origin xyz="${chassisLength/2} ${-2*sensorSpacing} ${wheelRadius/2}" rpy="0 ${sensorAngle} 0"/>
+    <parent link="chassis"/>
+    <child link="r_sensor_2"/>
+  </joint>
+  <link name="r_sensor_2">
+    <collision>
+      <origin xyz="0 0 0" rpy="0 ${sensorAngle} 0"/>
+      <geometry>
+	<box size="${sensorSize} ${sensorSize} ${sensorSize}"/>
+      </geometry>
+    </collision>
+    <visual>
+      <origin xyz="0 0 0" rpy="0 ${sensorAngle} 0"/>
+      <geometry>
+	<box size="${sensorSize} ${sensorSize} ${sensorSize}"/>
+      </geometry>
+      <material name="blue"/>
+    </visual>
+    <inertial>
+      <mass value="${cameraMass}" />
+      <origin xyz="0 0 0" rpy="0 0 0"/>
+      <box_inertia m="${cameraMass}" x="${sensorSize}" y="${sensorSize}" z="${sensorSize}" />
+    </inertial>
+  </link>
+<!--/////////////////////////////////////////////////////////////////-->
+  <joint name="left_sensor3" type="fixed">
+    <origin xyz="${chassisLength/2} ${3*sensorSpacing} ${wheelRadius/2}" rpy="0 ${sensorAngle} 0"/>
+    <parent link="chassis"/>
+    <child link="l_sensor_3"/>
+  </joint>
+  <link name="l_sensor_3">
+    <collision>
+      <origin xyz="0 0 0" rpy="0 ${sensorAngle} 0"/>
+      <geometry>
+	<box size="${sensorSize} ${sensorSize} ${sensorSize}"/>
+      </geometry>
+    </collision>
+    <visual>
+      <origin xyz="0 0 0" rpy="0 ${sensorAngle} 0"/>
+      <geometry>
+	<box size="${sensorSize} ${sensorSize} ${sensorSize}"/>
+      </geometry>
+      <material name="blue"/>
+    </visual>
+    <inertial>
+      <mass value="${cameraMass}" />
+      <origin xyz="0 0 0" rpy="0 0 0"/>
+      <box_inertia m="${cameraMass}" x="${sensorSize}" y="${sensorSize}" z="${sensorSize}" />
+    </inertial>
+  </link>
+<!--/////////////////////////////////////////////////////////////////-->
+  <joint name="right_sensor3" type="fixed">
+    <origin xyz="${chassisLength/2} ${-3*sensorSpacing} ${wheelRadius/2}" rpy="0 ${sensorAngle} 0"/>
+    <parent link="chassis"/>
+    <child link="r_sensor_3"/>
+  </joint>
+  <link name="r_sensor_3">
+    <collision>
+      <origin xyz="0 0 0" rpy="0 ${sensorAngle} 0"/>
+      <geometry>
+	<box size="${sensorSize} ${sensorSize} ${sensorSize}"/>
+      </geometry>
+    </collision>
+    <visual>
+      <origin xyz="0 0 0" rpy="0 ${sensorAngle} 0"/>
+      <geometry>
+	<box size="${sensorSize} ${sensorSize} ${sensorSize}"/>
+      </geometry>
+      <material name="blue"/>
+    </visual>
+    <inertial>
+      <mass value="${cameraMass}" />
+      <origin xyz="0 0 0" rpy="0 0 0"/>
+      <box_inertia m="${cameraMass}" x="${sensorSize}" y="${sensorSize}" z="${sensorSize}" />
+    </inertial>
+  </link>
+<!--/////////////////////////////////////////////////////////////////-->
+  <joint name="left_sensor4" type="fixed">
+    <origin xyz="${chassisLength/2} ${4*sensorSpacing} ${wheelRadius/2}" rpy="0 ${sensorAngle} 0"/>
+    <parent link="chassis"/>
+    <child link="l_sensor_4"/>
+  </joint>
+  <link name="l_sensor_4">
+    <collision>
+      <origin xyz="0 0 0" rpy="0 ${sensorAngle} 0"/>
+      <geometry>
+	<box size="${sensorSize} ${sensorSize} ${sensorSize}"/>
+      </geometry>
+    </collision>
+    <visual>
+      <origin xyz="0 0 0" rpy="0 ${sensorAngle} 0"/>
+      <geometry>
+	<box size="${sensorSize} ${sensorSize} ${sensorSize}"/>
+      </geometry>
+      <material name="blue"/>
+    </visual>
+    <inertial>
+      <mass value="${cameraMass}" />
+      <origin xyz="0 0 0" rpy="0 0 0"/>
+      <box_inertia m="${cameraMass}" x="${sensorSize}" y="${sensorSize}" z="${sensorSize}" />
+    </inertial>
+  </link>
+<!--/////////////////////////////////////////////////////////////////-->
+  <joint name="right_sensor4" type="fixed">
+    <origin xyz="${chassisLength/2} ${-4*sensorSpacing} ${wheelRadius/2}" rpy="0 ${sensorAngle} 0"/>
+    <parent link="chassis"/>
+    <child link="r_sensor_4"/>
+  </joint>
+  <link name="r_sensor_4">
+    <collision>
+      <origin xyz="0 0 0" rpy="0 ${sensorAngle} 0"/>
+      <geometry>
+	<box size="${sensorSize} ${sensorSize} ${sensorSize}"/>
+      </geometry>
+    </collision>
+    <visual>
+      <origin xyz="0 0 0" rpy="0 ${sensorAngle} 0"/>
+      <geometry>
+	<box size="${sensorSize} ${sensorSize} ${sensorSize}"/>
+      </geometry>
+      <material name="blue"/>
+    </visual>
+    <inertial>
+      <mass value="${cameraMass}" />
+      <origin xyz="0 0 0" rpy="0 0 0"/>
+      <box_inertia m="${cameraMass}" x="${sensorSize}" y="${sensorSize}" z="${sensorSize}" />
+    </inertial>
+  </link>
 </robot>

Commit message: changed sensor angle to point at the ground

File: Gazebo/catkin_ws/src/mybot_description/urdf/mybot.xacro (robot description, xacro)
@@ -16,5 +16,5 @@
   <xacro:property name="cameraAngle" value="20"/>
   <xacro:property name="sensorSize" value="0.01"/>
-  <xacro:property name="sensorAngle" value="45"/>
+  <xacro:property name="sensorAngle" value="${PI/2}"/>
   <xacro:property name="sensorSpacing" value="0.04"/>
   <xacro:include filename="$(find mybot_description)/urdf/mybot.gazebo" />

Commit message: Convolutional Net working

File: Gazebo/catkin_ws/src/mybot_description/urdf/mybot.xacro (robot description, xacro)
@@ -14,5 +14,5 @@
   <xacro:property name="cameraSize" value="0.05"/>
   <xacro:property name="cameraMass" value="0.1"/>
-  <xacro:property name="cameraAngle" value="20"/>
+  <xacro:property name="cameraAngle" value="1.22"/>
   <xacro:property name="sensorSize" value="0.01"/>
   <xacro:property name="sensorAngle" value="${PI/2}"/>
